File: projects/elektroniczna_klepsydra/elektroniczna_klepsydra.kicad_sch (KiCad schematic)
At the start: 29 parts, among them J1 +, J2 -, SW1 SW_Push, T1 BC548, T2 BC548, T3 BC548, T4 BC558, T5 BC548, T6 BC558, T7 BC558, Y1 3V

Commit message: finalize R1 for elektroniczna_klepsydra
Parts:
- J1, J2: symbol Custom_Generic:Conn_01x01 -> Custom_Generic:Conn_Point
- T1, T2, T3, T5: symbol Custom_Generic:NPN BJT -> Custom_Generic:NPN_BJT_CBE
- T4, T6, T7: symbol Custom_Generic:PNP BJT -> Custom_Generic:PNP_BJT_CBE
Changed lines of the file:
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@@
     (effects (font (size 1.524 1.524)) (justify left bottom))
   )
-  (symbol (lib_name "C_Polarized_1") (lib_id "Custom_Generic:C_Polarized") (at 175.26 91.44 270) (unit 1)
+  (symbol (lib_id "Custom_Generic:C_Polarized") (at 175.26 91.44 270) (unit 1)
     (in_bom yes) (on_board yes)
     (property "Reference" "C2" (id 0) (at 175.26 84.455 90)
@@
     (pin "2")
   )
-  (symbol (lib_id "Custom_Generic:PNP BJT") (at 167.005 75.565 0) (mirror x) (unit 1)
+  (symbol (lib_id "Custom_Generic:R") (at 108.585 130.175 0) (unit 1)
+    (in_bom yes) (on_board yes)
+    (property "Reference" "R1" (id 0) (at 110.49 128.27 0)
+      (effects (font (size 1.524 1.524)) (justify left))
+    )
+    (property "Value" "1MΩ" (id 1) (at 110.49 132.08 0)
+      (effects (font (size 1.524 1.524)) (justify left))
+    )
+    (property "Footprint" "VeeCad:AX1_1N" (id 2) (at 106.807 130.175 90)
+      (effects (font (size 1.27 1.27)) hide)
+    )
+    (property "Datasheet" "" (id 3) (at 108.585 130.175 0)
+      (effects (font (size 1.27 1.27)) hide)
+    )
+    (pin "1")
+    (pin "2")
+  )
+  (symbol (lib_id "Custom_Generic:PNP_BJT_CBE") (at 167.005 75.565 0) (mirror x) (unit 1)
     (in_bom yes) (on_board yes)
     (property "Reference" "T6" (id 0) (at 170.815 73.66 0)
@@
     (pin "1")
   )
-  (symbol (lib_id "Custom_Generic:Conn_01x01") (at 212.725 76.835 270) (mirror x) (unit 1)
+  (symbol (lib_id "Custom_Generic:Conn_Point") (at 212.725 76.835 270) (mirror x) (unit 1)
     (in_bom yes) (on_board yes)
     (property "Reference" "J2" (id 0) (at 210.185 75.565 90)
@@
     (pin "1")
   )
-  (symbol (lib_name "C_Polarized_2") (lib_id "Custom_Generic:C_Polarized") (at 191.77 68.58 0) (mirror y) (unit 1)
+  (symbol (lib_id "Custom_Generic:C_Polarized") (at 191.77 68.58 0) (mirror y) (unit 1)
     (in_bom yes) (on_board yes)
     (property "Reference" "C3" (id 0) (at 191.135 62.865 0)
@@
     (pin "1")
   )
-  (symbol (lib_id "Custom_Generic:R") (at 108.585 130.175 0) (unit 1)
-    (in_bom yes) (on_board yes)
-    (property "Reference" "R1" (id 0) (at 110.49 128.27 0)
-      (effects (font (size 1.524 1.524)) (justify left))
-    )
-    (property "Value" "1MΩ" (id 1) (at 110.49 132.08 0)
-      (effects (font (size 1.524 1.524)) (justify left))
-    )
-    (property "Footprint" "VeeCad:AX1_1N" (id 2) (at 106.807 130.175 90)
-      (effects (font (size 1.27 1.27)) hide)
-    )
-    (property "Datasheet" "" (id 3) (at 108.585 130.175 0)
-      (effects (font (size 1.27 1.27)) hide)
-    )
-    (pin "1")
-    (pin "2")
-  )
   (symbol (lib_id "Custom_Generic:D") (at 181.61 75.565 270) (unit 1)
     (in_bom yes) (on_board yes)
@@
     (pin "2")
   )
-  (symbol (lib_id "Custom_Generic:NPN BJT") (at 123.19 85.09 0) (unit 1)
+  (symbol (lib_id "Custom_Generic:NPN_BJT_CBE") (at 123.19 85.09 0) (unit 1)
     (in_bom yes) (on_board yes)
     (property "Reference" "T3" (id 0) (at 118.745 83.185 0)
@@
     (pin "2")
   )
-  (symbol (lib_id "Custom_Generic:NPN BJT") (at 140.335 120.015 0) (unit 1)
+  (symbol (lib_id "Custom_Generic:NPN_BJT_CBE") (at 140.335 120.015 0) (unit 1)
     (in_bom yes) (on_board yes)
     (property "Reference" "T2" (id 0) (at 144.145 118.11 0)
@@
     (pin "2")
   )
-  (symbol (lib_id "Custom_Generic:NPN BJT") (at 111.125 120.015 0) (mirror y) (unit 1)
+  (symbol (lib_id "Custom_Generic:NPN_BJT_CBE") (at 111.125 120.015 0) (mirror y) (unit 1)
     (in_bom yes) (on_board yes)
     (property "Reference" "T1" (id 0) (at 107.315 118.11 0)
@@
     (pin "3")
   )
-  (symbol (lib_id "Custom_Generic:PNP BJT") (at 198.12 91.44 0) (mirror x) (unit 1)
+  (symbol (lib_id "Custom_Generic:PNP_BJT_CBE") (at 198.12 91.44 0) (mirror x) (unit 1)
     (in_bom yes) (on_board yes)
     (property "Reference" "T7" (id 0) (at 201.93 89.535 0)
@@
     (pin "1")
   )
-  (symbol (lib_id "Custom_Generic:NPN BJT") (at 149.86 91.44 0) (mirror y) (unit 1)
+  (symbol (lib_id "Custom_Generic:NPN_BJT_CBE") (at 149.86 91.44 0) (mirror y) (unit 1)
     (in_bom yes) (on_board yes)
     (property "Reference" "T5" (id 0) (at 154.305 89.535 0)
@@
     (pin "1")
   )
-  (symbol (lib_id "Custom_Generic:Conn_01x01") (at 212.725 66.675 270) (unit 1)
+  (symbol (lib_id "Custom_Generic:Conn_Point") (at 212.725 66.675 270) (unit 1)
     (in_bom yes) (on_board yes)
     (property "Reference" "J1" (id 0) (at 213.995 69.215 0)
@@
     (pin "1")
   )
-  (symbol (lib_id "Custom_Generic:PNP BJT") (at 135.89 91.44 0) (mirror x) (unit 1)
+  (symbol (lib_id "Custom_Generic:PNP_BJT_CBE") (at 135.89 91.44 0) (mirror x) (unit 1)
     (in_bom yes) (on_board yes)
     (property "Reference" "T4" (id 0) (at 131.445 89.535 0)
@@
       (reference "J2") (unit 1) (value "-") (footprint "VeeCad:SIP1")
     )
-    (path "/61e20054-3617-4050-a267-0392cdaa1603"
+    (path "/21f4bd02-c635-4e92-872d-010e71376d5a"
       (reference "R1") (unit 1) (value "1MΩ") (footprint "VeeCad:AX1_1N")
     )

Commit message: elektroniczna_klepsydra_R2
Parts:
- removed C2: 4,7μF, VeeCad:RA1_2, symbol Custom_Generic:C_Polarized
- removed D3: 4148, VeeCad:AX1_1, symbol Custom_Generic:D
- removed T7: BC558, VeeCad:TO92, symbol Custom_Generic:PNP_BJT_CBE
- removed Y1: 3V, VeeCad:BUZR_12, symbol Custom_Generic:Buzzer_Magnetic_Active
- added C2: 1μF, VeeCad:RA2_4, symbol Custom_Generic:C
- added P1: 200k, symbol *Custom_Generic:P
- added R11, R16: 100kΩ, VeeCad:AX1_1N, symbol Custom_Generic:R
- added R14, R15, R17: 10kΩ, VeeCad:AX1_1N, symbol Custom_Generic:R
- added T7, T8: BC548, VeeCad:TO92, symbol Custom_Generic:NPN_BJT_CBE
- added T9: BC558, VeeCad:TO92, symbol Custom_Generic:PNP_BJT_CBE
- added Y1: Buzzer_Piezo_Active, symbol *Custom_Generic:Buzzer_Piezo_Active
- C1: value 1000μF -> 100μF
- R1: value 1MΩ -> 100kΩ
- R10: value 22kΩ -> 1MΩ
- R13: value 150Ω -> 100kΩ
Connections:
- net GNDD: now also C2.2, P1.3, R17.2, Y1.2; no longer R1.2
- net VCC: now also R13.1, R15.1, T9.3 (E)
- net at R10.2, R9.1, T6.1 (C): now also T7.3 (E), T8.3 (E)
- net at R1.1: now also R17.1, T9.1 (C), Y1.1; no longer T1.3 (E)
- net at R13.2: now also R14.1, T7.1 (C)
- new net: R15.2, R16.1, T8.1 (C)
- new net: R16.2, T9.2 (B)
- new net: C2.1, R1.2, R11.1
- new net: R14.2, T8.2 (B)
- new net: P1.1, P1.2, T1.3 (E)
- new net: R11.2, T7.2 (B)
Other:
- moved on the sheet: C1, C3, D1, D2, R10, R12, R2, R3, R4, R5, R6, R7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

Commit message: elektroniczna_klepsydra_R3
Parts:
- removed Y1: Buzzer_Piezo_Active, symbol *Custom_Generic:Buzzer_Piezo_Active
- added D3: 3V3, symbol *Custom_Generic:D_zener
- added R18: 10kΩ, VeeCad:AX1_1N, symbol Custom_Generic:R
- added T10: BC548, VeeCad:TO92, symbol Custom_Generic:NPN_BJT_CBE
- added Y1: Buzzer_Magnetic_Active, symbol *Custom_Generic:Buzzer_Magnetic_Active
Connections:
- net GNDD: now also D3.2 (A), Y1.2
- net VCC: now also T10.1 (C)
- net at R1.1, R17.1, T9.1 (C): now also R18.1
- new net: T10.3 (E), Y1.1
- new net: D3.1 (K), R18.2, T10.2 (B)
Other:
- moved on the sheet: C1, C2, C3, D1, D2, P1, R1, R10, R11, R12, R13, R14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
