File: projects/smt_adapters/so16__dip16/panel.kicad_pcb (KiCad board)
At the start: 2 copper layers, 84.9 x 87.1 mm, 28 parts, among them U1 DIP-16_W7.62mm, U2 SOIC-16W_7.5x10.3mm_P1.27mm

Commit message: just making sure everything's there
Parts:
- removed the U1 at (115.6, 117.9)
- removed the U1 at (115.6, 142.8)
- removed the U1 at (151.0, 105.5)
- removed the U1 at (151.0, 117.9)
- removed the U1 at (115.6, 68.1)
- removed the U1 at (151.0, 130.4)
- removed the U1 at (151.0, 68.1)
- removed the U1 at (115.6, 93.0)
- removed the U1 at (151.0, 142.8)
- removed the U1 at (151.0, 80.6)
- removed the U1 at (151.0, 93.0)
- removed the U1 at (115.6, 80.6)
- removed the U1 at (115.6, 130.4)
- removed the U1 at (115.6, 105.5)
- removed the U2 at (177.1, 101.7)
- removed the U2 at (141.6, 76.8)
- removed the U2 at (177.1, 64.3)
- removed the U2 at (177.1, 126.6)
- removed the U2 at (141.6, 89.2)
- removed the U2 at (177.1, 89.2)
- removed the U2 at (141.6, 64.3)
- removed the U2 at (141.6, 126.6)
- removed the U2 at (177.1, 76.8)
- removed the U2 at (177.1, 114.1)
- removed the U2 at (141.6, 139.0)
- removed the U2 at (141.6, 114.1)
- removed the U2 at (141.6, 101.7)
- removed the U2 at (177.1, 139.0)
- added U1: DIP-16_W7.62mm, Package_DIP:DIP-16_W7.62mm, F.Cu at (115.6, 92.3)
- added U1: DIP-16_W7.62mm, Package_DIP:DIP-16_W7.62mm, F.Cu at (151.0, 104.7)
- added U1: DIP-16_W7.62mm, Package_DIP:DIP-16_W7.62mm, F.Cu at (151.0, 42.5)
- added U1: DIP-16_W7.62mm, Package_DIP:DIP-16_W7.62mm, F.Cu at (115.6, 42.5)
- added U1: DIP-16_W7.62mm, Package_DIP:DIP-16_W7.62mm, F.Cu at (115.6, 79.8)
- added U1: DIP-16_W7.62mm, Package_DIP:DIP-16_W7.62mm, F.Cu at (151.0, 92.3)
- added U1: DIP-16_W7.62mm, Package_DIP:DIP-16_W7.62mm, F.Cu at (151.0, 67.4)
- added U1: DIP-16_W7.62mm, Package_DIP:DIP-16_W7.62mm, F.Cu at (151.0, 79.8)
- added U1: DIP-16_W7.62mm, Package_DIP:DIP-16_W7.62mm, F.Cu at (151.0, 54.9)
- added U1: DIP-16_W7.62mm, Package_DIP:DIP-16_W7.62mm, F.Cu at (151.0, 30.0)
- added U1: DIP-16_W7.62mm, Package_DIP:DIP-16_W7.62mm, F.Cu at (115.6, 54.9)
- added U1: DIP-16_W7.62mm, Package_DIP:DIP-16_W7.62mm, F.Cu at (115.6, 30.0)
- added U1: DIP-16_W7.62mm, Package_DIP:DIP-16_W7.62mm, F.Cu at (115.6, 104.7)
- added U1: DIP-16_W7.62mm, Package_DIP:DIP-16_W7.62mm, F.Cu at (115.6, 67.4)
- added U2: SOIC-16W_7.5x10.3mm_P1.27mm, Package_SO:SOIC-16W_7.5x10.3mm_P1.27mm, F.Cu at (141.6, 38.7)
- added U2: SOIC-16W_7.5x10.3mm_P1.27mm, Package_SO:SOIC-16W_7.5x10.3mm_P1.27mm, F.Cu at (177.1, 76.0)
- added U2: SOIC-16W_7.5x10.3mm_P1.27mm, Package_SO:SOIC-16W_7.5x10.3mm_P1.27mm, F.Cu at (177.1, 51.1)
- added U2: SOIC-16W_7.5x10.3mm_P1.27mm, Package_SO:SOIC-16W_7.5x10.3mm_P1.27mm, F.Cu at (141.6, 76.0)
- added U2: SOIC-16W_7.5x10.3mm_P1.27mm, Package_SO:SOIC-16W_7.5x10.3mm_P1.27mm, F.Cu at (141.6, 51.1)
- added U2: SOIC-16W_7.5x10.3mm_P1.27mm, Package_SO:SOIC-16W_7.5x10.3mm_P1.27mm, F.Cu at (141.6, 100.9)
- added U2: SOIC-16W_7.5x10.3mm_P1.27mm, Package_SO:SOIC-16W_7.5x10.3mm_P1.27mm, F.Cu at (177.1, 38.7)
- added U2: SOIC-16W_7.5x10.3mm_P1.27mm, Package_SO:SOIC-16W_7.5x10.3mm_P1.27mm, F.Cu at (141.6, 88.5)
- added U2: SOIC-16W_7.5x10.3mm_P1.27mm, Package_SO:SOIC-16W_7.5x10.3mm_P1.27mm, F.Cu at (141.6, 26.2)
- added U2: SOIC-16W_7.5x10.3mm_P1.27mm, Package_SO:SOIC-16W_7.5x10.3mm_P1.27mm, F.Cu at (177.1, 63.6)
- added U2: SOIC-16W_7.5x10.3mm_P1.27mm, Package_SO:SOIC-16W_7.5x10.3mm_P1.27mm, F.Cu at (177.1, 26.2)
- added U2: SOIC-16W_7.5x10.3mm_P1.27mm, Package_SO:SOIC-16W_7.5x10.3mm_P1.27mm, F.Cu at (141.6, 63.6)
- added U2: SOIC-16W_7.5x10.3mm_P1.27mm, Package_SO:SOIC-16W_7.5x10.3mm_P1.27mm, F.Cu at (177.1, 88.5)
- added U2: SOIC-16W_7.5x10.3mm_P1.27mm, Package_SO:SOIC-16W_7.5x10.3mm_P1.27mm, F.Cu at (177.1, 100.9)
Other:
- board text removed: "foresterr"
