File: projects/smt_adapters/so16__dip16/so16__dip16.kicad_pcb (KiCad board)
At the start: 2 copper layers, 35.4 x 12.4 mm, 2 parts, among them U1 DIP-16_W7.62mm, U2 SOIC-16W_7.5x10.3mm_P1.27mm

Commit message: just making sure everything's there
Other:
- board text removed: "foresterr"
